File: V2_1/ClockV2_1/ClockV2_1.kicad_sch (KiCad schematic)
At the start: 0 parts

Commit message: started layout
Parts:
- added U1: NUCLEO-L432KC, NUCLEO-L432KC:MODULE_NUCLEO-L432KC, symbol NUCLEO-L432KC:NUCLEO-L432KC
Other:
- added sheet Display driver and io (Display_driver.kicad_sch)
- added sheet Front panel (untitled.kicad_sch)
