File: V2_1/ClockV2_1/ClockV2_1.kicad_sch (KiCad schematic)
At the start: 1 part, among them U1 NUCLEO-L432KC

Commit message: aaaaaah i forgot about github
new software repo
Parts:
- added C105: 15p, Capacitor_SMD:C_0603_1608Metric, symbol Device:C
- added C107, C109: 150p, Capacitor_SMD:C_0603_1608Metric, symbol Device:C
- added H101, H102, H103, H104: MountingHole_Pad, MountingHole:MountingHole_3.2mm_M3_DIN965_Pad, symbol Mechanical:MountingHole_Pad
- added J101: Conn_Coaxial, Connector_Coaxial:SMA_Amphenol_132289_EdgeMount, symbol Connector:Conn_Coaxial
- added J103, J104: Conn_02x04_Odd_Even, Connector_PinSocket_2.54mm:PinSocket_2x04_P2.54mm_Vertical, symbol Connector_Generic:Conn_02x04_Odd_Even
- added J105: DIN41612_02x16_AC_EvenPins, Connector_DIN:DIN41612_C_2x16_Male_Horizontal_THT, symbol Connector:DIN41612_02x16_AC_EvenPins
- added JP2, JP3: SolderJumper_2_Open, Jumper:SolderJumper-2_P1.3mm_Open_RoundedPad1.0x1.5mm, symbol Jumper:SolderJumper_2_Open
- added L101: 8.4u 2%, Inductor_SMD:L_0603_1608Metric, symbol Device:L
- added L102: 620n 2%, Inductor_SMD:L_1008_2520Metric, symbol Device:L
- added R107: 1k, Resistor_SMD:R_0805_2012Metric, symbol Device:R
- added R111: 330R, Resistor_SMD:R_0805_2012Metric, symbol Device:R
- U1: footprint NUCLEO-L432KC:MODULE_NUCLEO-L432KC -> ClockV2_1:MODULE_NUCLEO-L432KC; now left out of the parts list
Connections:
- net Thermistor: now reaches U1.CN4_10 (PA3)
- net Thermistor: now also J103.1 (Pin_1)
- net light_sense: now reaches U1.CN4_11 (PA1)
- net Xtal: now reaches U1.CN4_12 (PA0)
- net Xtal: now also C109.1, J103.5 (Pin_5), JP3.2 (B)
- net +3.3VA: now reaches U1.CN4_13 (AREF)
- net +3.3VA: now also J104.3 (Pin_3)
- net +3.3V: now reaches U1.CN4_14 (+3V3)
- net GND: now reaches U1.CN4_2 (GND_CN4)
- net GND: now also U1.CN3_4 (GND_CN3), C107.2, H101.1, H102.1, H103.1, H104.1, J101.2 (Ext), J103.3 (Pin_3), J103.4 (Pin_4), J103.6 (Pin_6), J103.7 (Pin_7), J103.8 (Pin_8), J104.2 (Pin_2), J104.4 (Pin_4), J104.6 (Pin_6), J104.8 (Pin_8), J105.a12 (Pin_a12), J105.a20 (Pin_a20), J105.a24 (Pin_a24), J105.a4 (Pin_a4), J105.c12 (Pin_c12), J105.c24 (Pin_c24), J105.c4 (Pin_c4), L102.2, R107.2
- net +5V: now reaches U1.CN4_4 (+5V)
- net +5V: now also J104.5 (Pin_5), J104.7 (Pin_7)
- net 1Hz: now reaches U1.CN4_5 (PA2)
- net 1Hz: now also JP2.2 (B)
- net I2C SCL: now reaches U1.CN3_1 (PA9)
- net I2C SCL: now also J105.a16 (Pin_a16)
- net LED: now reaches U1.CN3_10 (PC14)
- net Button: now reaches U1.CN3_11 (PC15)
- net I2C SDA: now reaches U1.CN3_2 (PA10)
- net I2C SDA: now also J105.a18 (Pin_a18)
- net Ock: now reaches U1.CN3_5 (PA12)
- net OE: now reaches U1.CN3_6 (PB0)
- net sck: now reaches U1.CN3_7 (PB7)
- net SDA: now reaches U1.CN3_8 (PB6)
- net Heater_PWM: now reaches U1.CN3_9 (PB1)
- net Heater_PWM: now also J103.2 (Pin_2)
- new net: J105.c20 (Pin_c20), JP2.1 (A)
- new net: C105.1, C107.1, L102.1, R111.2
- new net: C105.2, L101.1
- new net: C109.2, R111.1
- new net: J105.c22 (Pin_c22), JP3.1 (A)
- new net +12P: J105.a2 (Pin_a2), J105.c2 (Pin_c2)
- new net 16MHz sine: J101.1 (In), L101.2, R107.1
- no-connect marks 0 -> 19
Other:
- added sheet Battery and power (Power_and_batt.kicad_sch)
- added sheet Oven and heater (oven.kicad_sch)
- sheet Display driver and io ports: added ORClk, OutEn, Sclk, SerData; removed none
- title: (none) -> Clock Card
- moved on the sheet: U1A, U1B

Commit message: updates
Connections:
- net 1Hz: no longer names the net of U1.CN4_5 (PA2)
- net 1Hz: no longer JP2.2 (B)
- new net 1pps: JP2.2 (B)
Changed lines of the file:
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@@
-		)
-	)
-	(label "1Hz"
-		(at 52.07 110.49 0)
-		(effects
-			(font
-				(size 1.27 1.27)
-			)
-			(justify left bottom)
 		)
 	)
@@
 		)
 	)
-	(label "1Hz"
-		(at 133.35 85.09 180)
-		(effects
-			(font
-				(size 1.27 1.27)
-			)
-			(justify right bottom)
-		)
-	)
 	(label "Xtal"
 		(at 179.07 30.48 180)
@@
 		)
 	)
+	(global_label "1pps"
+		(shape input)
+		(at 130.81 105.41 180)
+		(fields_autoplaced yes)
+		(effects
+			(font
+				(size 1.27 1.27)
+			)
+			(justify right)
+		)
+		(property "Intersheetrefs" "${INTERSHEET_REFS}"
+			(at 123.2892 105.41 0)
+			(effects
+				(font
+					(size 1.27 1.27)
+				)
+				(justify right)
+				(hide yes)
+			)
+		)
+	)
 	(global_label "Button"
 		(shape input)
@@
 				(hide yes)
 			)
+		)
+	)
+	(global_label "1pps"
+		(shape input)
+		(at 52.07 110.49 0)
+		(fields_autoplaced yes)
+		(effects
+			(font
+				(size 1.27 1.27)
+			)
+			(justify left)
+		)
+		(property "Intersheetrefs" "${INTERSHEET_REFS}"
+			(at 59.5908 110.49 0)
+			(effects
+				(font
+					(size 1.27 1.27)
+				)
+				(justify left)
+				(hide yes)
+			)
