File: V2_1/ClockV2_1/_autosave-ClockV2_1.kicad_sch (KiCad schematic)
At the start: 8 parts, among them J103 Conn_02x04_Odd_Even, J104 Conn_02x04_Odd_Even, J105 DIN41612_02x16_AC_EvenPins, U1 NUCLEO-L432KC

Commit message: aaaaaah i forgot about github
new software repo
Parts:
- added C105: 15p, Capacitor_SMD:C_0603_1608Metric, symbol Device:C
- added C107, C109: 150p, Capacitor_SMD:C_0603_1608Metric, symbol Device:C
- added J101: Conn_Coaxial, Connector_Coaxial:SMA_Amphenol_132289_EdgeMount, symbol Connector:Conn_Coaxial
- added JP2, JP3: SolderJumper_2_Open, Jumper:SolderJumper-2_P1.3mm_Open_RoundedPad1.0x1.5mm, symbol Jumper:SolderJumper_2_Open
- added L101: 8.4u 2%, Inductor_SMD:L_0603_1608Metric, symbol Device:L
- added L102: 620n 2%, Inductor_SMD:L_1008_2520Metric, symbol Device:L
- added R107: 1k, Resistor_SMD:R_0805_2012Metric, symbol Device:R
- added R111: 330R, Resistor_SMD:R_0805_2012Metric, symbol Device:R
- H101, H102, H104: now left out of the parts list
- U1: footprint NUCLEO-L432KC:MODULE_NUCLEO-L432KC -> ClockV2_1:MODULE_NUCLEO-L432KC; now left out of the parts list
Connections:
- net GND: now also C107.2, J101.2 (Ext), L102.2, R107.2
- net Heater_PWM: now also U1.CN3_9 (PB1)
- net Thermistor: now also U1.CN4_10 (PA3)
- net Xtal: now also J103.5 (Pin_5), C109.1, JP3.2 (B)
- net light_sense: now reaches U1.CN4_11 (PA1)
- net I2C SCL: now reaches J105.a16 (Pin_a16)
- net I2C SCL: now also U1.CN3_1 (PA9)
- net I2C SDA: now reaches J105.a18 (Pin_a18)
- net I2C SDA: now also U1.CN3_2 (PA10)
- net LED: now reaches U1.CN3_10 (PC14)
- net Button: now reaches U1.CN3_11 (PC15)
- net Ock: now reaches U1.CN3_5 (PA12)
- net OE: now reaches U1.CN3_6 (PB0)
- net sck: now reaches U1.CN3_7 (PB7)
- net SDA: now reaches U1.CN3_8 (PB6)
- net 16MHz clk: no longer names the net of J105.c22 (Pin_c22)
- net 16MHz clk: now also JP3.1 (A)
- net 1Hz: no longer names the net of J105.c20 (Pin_c20)
- net 1Hz: now also JP2.1 (A)
- new net: C105.1, C107.1, L102.1, R111.2
- new net: C105.2, L101.1
- new net: C109.2, R111.1
- new net 16MHz sine: J101.1 (In), L101.2, R107.1
- new net 1pps: JP2.2 (B)
- no-connect marks 4 -> 19
Other:
- sheet Display driver and io ports: added ORClk, OutEn, Sclk, SerData; removed none
- sheet Oven and heater ports: added none; removed Heater_PWM, Thermistor, XTAL1
- title: (none) -> Clock Card
