File: V2_1/ClockV2_1/Display_driver.kicad_sch (KiCad schematic)
At the start: 0 parts

Commit message: aaaaaah i forgot about github
new software repo
Parts:
- added C11, C12, C13: 1u, Capacitor_SMD:C_0805_2012Metric, symbol Device:C
- added J302: Conn_02x04_Odd_Even, Connector_PinHeader_2.54mm:PinHeader_2x04_P2.54mm_Horizontal, symbol Connector_Generic:Conn_02x04_Odd_Even
- added J303: Conn_02x06_Odd_Even, Connector_PinHeader_2.54mm:PinHeader_2x06_P2.54mm_Horizontal, symbol Connector_Generic:Conn_02x06_Odd_Even
- added JP4, JP5, JP6, JP7, JP8, JP9: SolderJumper_2_Open, Jumper:SolderJumper-2_P1.3mm_Open_RoundedPad1.0x1.5mm, symbol Jumper:SolderJumper_2_Open
- added R301, R302, R303, R304, R305, R306, R307, R308, R310, R318: 150, Resistor_SMD:R_0805_2012Metric, symbol Device:R
- added U301, U302, U303: 74HC595, Package_SO:SOIC-16_3.9x9.9mm_P1.27mm, symbol 74xx:74HC595
- added j304: Conn_01x04, Connector_PinHeader_2.54mm:PinHeader_1x04_P2.54mm_Horizontal, symbol Connector_Generic:Conn_01x04
Connections:
- new net: JP9.1 (A), U303.6 (QG)
- new net: R302.1, U301.1 (QB)
- new net: R303.1, U301.2 (QC)
- new net: JP4.1 (A), U302.15 (QA)
- new net: R305.1, U301.4 (QE)
- new net: R318.1, U302.4 (QE)
- new net: JP5.1 (A), U302.2 (QC)
- new net: R310.2, U302.5 (QF)
- new net: U302.9 (QH'), U303.14 (SER)
- new net: JP8.1 (A), U303.4 (QE)
- new net: R307.1, U301.6 (QG)
- new net: JP6.1 (A), U303.15 (QA)
- new net: JP7.1 (A), U303.2 (QC)
- new net: U301.14 (SER), U303.9 (QH')
- new net: R301.1, U301.15 (QA)
- new net: R304.1, U301.3 (QD)
- new net: R306.1, U301.5 (QF)
- new net: R308.1, U301.7 (QH)
- new net +3.3V: C11.1, C12.1, C13.1, J303.8 (Pin_8), U301.10 (~{SRCLR}), U301.16 (VCC), U302.10 (~{SRCLR}), U302.16 (VCC), U303.10 (~{SRCLR}), U303.16 (VCC)
- new net +5V: j304.3 (Pin_3)
- new net 1PPS: J303.5 (Pin_5)
- new net A1: J303.4 (Pin_4), JP4.2 (B), U302.1 (QB)
- new net A2: J303.2 (Pin_2), JP5.2 (B), U302.3 (QD)
- new net A5: J303.9 (Pin_9), JP9.2 (B), U303.7 (QH)
- new net A6: J303.11 (Pin_11), JP8.2 (B), U303.5 (QF)
- new net A7: J303.12 (Pin_12), JP7.2 (B), U303.3 (QD)
- new net A8: J303.10 (Pin_10), JP6.2 (B), U303.1 (QB)
- new net Button: J303.7 (Pin_7)
- new net GND: C11.2, C12.2, C13.2, J303.3 (Pin_3), J303.6 (Pin_6), U301.13 (~{OE}), U301.8 (GND), U302.8 (GND), U303.8 (GND)
- new net LED: j304.1 (Pin_1)
- new net LED2: J303.1 (Pin_1), R318.2
- new net LED3: R310.1, j304.2 (Pin_2)
- new net ORClk: U301.12 (RCLK), U302.12 (RCLK), U303.12 (RCLK)
- new net OutEn: U302.13 (~{OE}), U303.13 (~{OE})
- new net Sclk: U301.11 (SRCLK), U302.11 (SRCLK), U303.11 (SRCLK)
- new net SerData: U302.14 (SER)
- new net a: J302.2 (Pin_2), R307.2
- new net b: J302.1 (Pin_1), R306.2
- new net c: J302.5 (Pin_5), R304.2
- new net d: J302.8 (Pin_8), R302.2
- new net dp: J302.7 (Pin_7), R303.2
- new net e: J302.6 (Pin_6), R301.2
- new net f: J302.4 (Pin_4), R308.2
- new net g: J302.3 (Pin_3), R305.2
- new net light_sense: j304.4 (Pin_4)
- no-connect marks 0 -> 2

Commit message: updates
Connections:
- net 1PPS renamed 1pps
Changed lines of the file:
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@@
-		)
-	)
-	(label "1PPS"
-		(at 193.04 99.06 0)
-		(effects
-			(font
-				(size 1.27 1.27)
-			)
-			(justify left bottom)
 		)
 	)
@@
 			(effects
 				(font
+					(size 1.27 1.27)
+				)
+				(justify left)
+				(hide yes)
+			)
+		)
+	)
+	(global_label "1pps"
+		(shape input)
+		(at 193.04 99.06 0)
+		(fields_autoplaced yes)
+		(effects
+			(font
+				(size 1.27 1.27)
+			)
+			(justify left)
+		)
+		(property "Intersheetrefs" "${INTERSHEET_REFS}"
+			(at 200.5608 99.06 0)
+			(effects
+				(font
