File: V2_1/ClockV2_1/untitled.kicad_sch (KiCad schematic)
At the start: 0 parts

Commit message: aaaaaah i forgot about github
new software repo
Parts:
- added D301, D302: RED, LED_SMD:LED_0805_2012Metric, symbol Device:LED
- added D304: GRN, LED_SMD:LED_0805_2012Metric, symbol Device:LED
- added DS401: LTD-4608JR, LTD_4608JR:LTD-4608JR_LTO, symbol 2025-07-31_16-04-08:LTD-4608JR
- added DS402: TDCR1060M, TDCR1060M:DISPLAY_TDCR1060M, symbol TDCR1060M:TDCR1060M
- added J401: Conn_01x04, Connector_PinHeader_2.54mm:PinHeader_1x04_P2.54mm_Vertical, symbol Connector_Generic:Conn_01x04
- added J402: Conn_02x04_Odd_Even, Connector_PinHeader_2.54mm:PinHeader_2x04_P2.54mm_Vertical_SMD, symbol Connector_Generic:Conn_02x04_Odd_Even
- added J403: Conn_02x06_Odd_Even, Connector_PinHeader_2.54mm:PinHeader_2x06_P2.54mm_Vertical_SMD, symbol Connector_Generic:Conn_02x06_Odd_Even
- added R309: LDR03, OptoDevice:R_LDR_5.1x4.3mm_P3.4mm_Vertical, symbol Sensor_Optical:LDR03
- added R311, R312: 1k, Resistor_SMD:R_0805_2012Metric, symbol Device:R
- added R313, R314, R315: 330R, Resistor_SMD:R_0805_2012Metric, symbol Device:R
- added R317: 150, Resistor_SMD:R_0805_2012Metric, symbol Device:R
- added SW301: SW_Push, Button_Switch_THT:SW_PUSH_6mm_H4.3mm, symbol Switch:SW_Push
Connections:
- new net: R313.1, R315.2
- new net: D301.2 (A), R313.2
- new net: D304.2 (A), R317.1
- new net: D302.2 (A), R314.2
- new net +3.3V: J403.8 (Pin_8), R312.1, R314.1
- new net +3.3VA: R311.1
- new net +5V: J401.3 (Pin_3), R315.1
- new net A1: DS401.9, J403.4 (Pin_4)
- new net A2: DS401.4, J403.2 (Pin_2)
- new net A5: DS402.1, J403.9 (Pin_9)
- new net A6: DS402.2, J403.11 (Pin_11)
- new net A7: DS402.6, J403.12 (Pin_12)
- new net A8: DS402.8, J403.10 (Pin_10)
- new net Button: J403.7 (Pin_7), R312.2, SW301.1
- new net GND: D301.1 (K), D302.1 (K), D304.1 (K), DS402.10, DS402.4, J403.3 (Pin_3), J403.6 (Pin_6), R309.2, SW301.2
- new net LED1: J401.1 (Pin_1), R317.2
- new net LED2: DS402.9, J401.2 (Pin_2), J403.1 (Pin_1)
- new net LED3: DS402.12, J403.5 (Pin_5)
- new net a: DS401.10, DS402.14, J402.2 (Pin_2)
- new net b: DS401.8, DS402.16, J402.1 (Pin_1)
- new net c: DS401.1, DS402.13, J402.5 (Pin_5)
- new net d: DS401.5, DS402.3, J402.8 (Pin_8)
- new net dp: DS401.2, DS402.7, J402.7 (Pin_7)
- new net e: DS401.3, DS402.5, J402.6 (Pin_6)
- new net f: DS401.6, DS402.11, J402.4 (Pin_4)
- new net g: DS401.7, DS402.15, J402.3 (Pin_3)
- new net light_sense: J401.4 (Pin_4), R309.1, R311.2

Commit message: updates
Parts:
- added D6: GRN, LED_SMD:LED_0805_2012Metric, symbol Device:LED
- added R6: 150, Resistor_SMD:R_0805_2012Metric, symbol Device:R
Connections:
- net GND: now also D6.1 (K)
- net LED2: no longer J401.2 (Pin_2)
- net LED3: now also J401.2 (Pin_2), R6.2; no longer DS402.12, J403.5 (Pin_5)
- new net: D6.2 (A), R6.1
- new net Colon: DS402.12
- new net colon: J403.5 (Pin_5)
Changed lines of the file:
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@@
+		)
+	)
+	(wire
+		(pts
+			(xy 241.3 134.62) (xy 237.49 134.62)
+		)
+		(stroke
+			(width 0)
+			(type default)
+		)
+	)
+	(wire
+		(pts
+			(xy 248.92 134.62) (xy 257.81 134.62)
+		)
+		(stroke
+			(width 0)
+			(type default)
 		)
 	)
@@
 		)
 	)
-	(label "LED3"
+	(label "Colon"
 		(at 156.21 146.05 0)
 		(effects
@@
 		)
 	)
-	(label "LED3"
+	(label "colon"
 		(at 58.42 111.76 0)
 		(effects
@@
 		)
 	)
-	(label "LED2"
+	(label "LED3"
 		(at 55.88 64.77 0)
 		(effects
@@
 			)
 			(justify left bottom)
+		)
+	)
+	(label "LED3"
+		(at 237.49 134.62 180)
+		(effects
+			(font
+				(size 1.27 1.27)
+			)
+			(justify right bottom)
 		)
 	)
@@
 	)
 	(symbol
+		(lib_id "power:GND")
+		(at 265.43 134.62 90)
+		(mirror x)
+		(unit 1)
+		(exclude_from_sim no)
+		(in_bom yes)
+		(on_board yes)
+		(dnp no)
+		(fields_autoplaced yes)
+		(property "Reference" "#PWR034"
+			(at 271.78 134.62 0)
+			(effects
+				(font
+					(size 1.27 1.27)
+				)
+				(hide yes)
+			)
+		)
+		(property "Value" "GND"
+			(at 270.51 134.62 0)
+			(effects
+				(font
+					(size 1.27 1.27)
+				)
+			)
+		)
+		(property "Footprint" ""
+			(at 265.43 134.62 0)
+			(effects
+				(font
+					(size 1.27 1.27)
+				)
+				(hide yes)
+			)
+		)
+		(property "Datasheet" ""
+			(at 265.43 134.62 0)
+			(effects
+				(font
+					(size 1.27 1.27)
+				)
+				(hide yes)
+			)
+		)
+		(property "Description" ""
+			(at 265.43 134.62 0)
+			(effects
+				(font
+					(size 1.27 1.27)
+				)
+			)
+		)
+		(pin "1"
+		)
+		(instances
+			(project "ClockV2_1"
+				(path "/7fcba237-8ca3-4071-83d7-ca8ca4007a89/b0fdcedf-8bbd-4382-ac8d-4d3cebb09152"
+					(reference "#PWR034")
+					(unit 1)
+				)
+			)
+		)
+	)
+	(symbol
 		(lib_id "Device:R")
 		(at 260.35 45.72 0)
@@
 	(symbol
 		(lib_id "Device:R")
+		(at 245.11 134.62 270)
+		(mirror x)
+		(unit 1)
+		(exclude_from_sim no)
+		(in_bom yes)
+		(on_board yes)
+		(dnp no)
+		(fields_autoplaced yes)
+		(property "Reference" "R6"
+			(at 244.475 137.16 0)
+			(effects
+				(font
+					(size 1.27 1.27)
+				)
+				(justify right)
+			)
+		)
+		(property "Value" "150"
+			(at 247.015 137.16 0)
+			(effects
+				(font
+					(size 1.27 1.27)
+				)
+				(justify right)
+			)
+		)
+		(property "Footprint" "Resistor_SMD:R_0805_2012Metric"
+			(at 245.11 136.398 90)
+			(effects
+				(font
+					(size 1.27 1.27)
+				)
+				(hide yes)
+			)
+		)
+		(property "Datasheet" "~"
+			(at 245.11 134.62 0)
+			(effects
+				(font
+					(size 1.27 1.27)
+				)
+				(hide yes)
+			)
+		)
+		(property "Description" ""
+			(at 245.11 134.62 0)
+			(effects
+				(font
+					(size 1.27 1.27)
+				)
+			)
+		)
+		(pin "1"
+		)
+		(pin "2"
+		)
+		(instances
+			(project "ClockV2_1"
+				(path "/7fcba237-8ca3-4071-83d7-ca8ca4007a89/b0fdcedf-8bbd-4382-ac8d-4d3cebb09152"
+					(reference "R6")
+					(unit 1)
+				)
+			)
+		)
+	)
+	(symbol
+		(lib_id "Device:R")
 		(at 260.35 74.93 0)
 		(mirror y)
@@
 					(unit 1)
 				)
+			)
+		)
+	)
+	(symbol
+		(lib_id "Device:LED")
+		(at 261.62 134.62 0)
+		(mirror y)
+		(unit 1)
+		(exclude_from_sim no)
+		(in_bom yes)
+		(on_board yes)
+		(dnp no)
+		(property "Reference" "D6"
+			(at 264.795 142.24 0)
+			(effects
+				(font
+					(size 1.27 1.27)
+				)
+			)
+		)
+		(property "Value" "GRN"
+			(at 265.43 139.7 0)
+			(effects
+				(font
+					(size 1.27 1.27)
+				)
+			)
+		)
+		(property "Footprint" "LED_SMD:LED_0805_2012Metric"
+			(at 261.62 134.62 0)
+			(effects
+				(font
+					(size 1.27 1.27)
+				)
+				(hide yes)
+			)
+		)
+		(property "Datasheet" "~"
+			(at 261.62 134.62 0)
+			(effects
+				(font
+					(size 1.27 1.27)
+				)
+				(hide yes)
+			)
+		)
+		(property "Description" ""
+			(at 261.62 134.62 0)
+			(effects
+				(font
+					(size 1.27 1.27)
+				)
+			)
+		)
+		(pin "1"
+		)
+		(pin "2"
+		)
+		(instances
+			(project "ClockV2_1"
+				(path "/7fcba237-8ca3-4071-83d7-ca8ca4007a89/b0fdcedf-8bbd-4382-ac8d-4d3cebb09152"
+					(reference "D6")
+					(unit 1)
+				)
