File: V2_0/7_seg_display.kicad_sch (KiCad schematic)
At the start: 38 parts, among them J301 Conn_01x04, J302 Conn_02x04_Odd_Even, J303 Conn_02x06_Odd_Even, J304 Conn_01x04, J402 Conn_02x04_Odd_Even, J403 Conn_02x06_Odd_Even, SW301 SW_Push, U301 74HC595, U302 74HC595, U303 74HC595

Commit message: aaaaaah i forgot about github
new software repo
Connections:
- net +3.3V: now also J303.8 (Pin_8); no longer J303.7 (Pin_7)
- net 1PPS: now also J303.5 (Pin_5); no longer J303.6 (Pin_6)
- net A1: now also J303.4 (Pin_4); no longer J303.3 (Pin_3)
- net A2: now also J303.2 (Pin_2); no longer J303.1 (Pin_1)
- net A5: now also J303.9 (Pin_9); no longer J303.10 (Pin_10)
- net A6: now also J303.11 (Pin_11); no longer J303.12 (Pin_12)
- net A7: now also J303.12 (Pin_12); no longer J303.11 (Pin_11)
- net A8: now also J303.10 (Pin_10); no longer J303.9 (Pin_9)
- net Button: now also J303.7 (Pin_7); no longer J303.8 (Pin_8)
- net GND: now also J303.3 (Pin_3), J303.6 (Pin_6); no longer J303.4 (Pin_4), J303.5 (Pin_5)
- net LED2: now also J303.1 (Pin_1); no longer J303.2 (Pin_2)
Changed lines of the file:
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@@
 	(symbol
 		(lib_id "Connector_Generic:Conn_02x06_Odd_Even")
-		(at 210.82 129.54 0)
+		(at 213.36 129.54 0)
+		(mirror y)
 		(unit 1)
 		(exclude_from_sim no)
@@
 		(on_board yes)
 		(dnp no)
-		(fields_autoplaced yes)
 		(property "Reference" "J303"
 			(at 212.09 119.38 0)
@@
 		)
 		(property "Footprint" "Connector_PinHeader_2.54mm:PinHeader_2x06_P2.54mm_Horizontal"
-			(at 210.82 129.54 0)
+			(at 213.36 129.54 0)
 			(effects
 				(font
@@
 		)
 		(property "Datasheet" "~"
-			(at 210.82 129.54 0)
+			(at 213.36 129.54 0)
 			(effects
 				(font
@@
 		)
 		(property "Description" ""
-			(at 210.82 129.54 0)
+			(at 213.36 129.54 0)
 			(effects
 				(font
